File: Aeroneers/CAD Files/projects/FSAE CONTROLLER/FSAE_CONTROLLER_DEUTSCH.sch (EAGLE design)
At the start: 23 parts, among them IC1 MPU-9250, IC2 R-783.3-1.0, U1 DUAL-OPTOISOLATOR_SOIC8

Commit message: End of semester commit
Parts:
- added F1: 1812L050, polyfuse-smd_10:1812L050
- J1: value (none) -> DTM13-12PA-R008; device SparkFun-Connectors:CONN_063.5MM-6 -> DTM13-12PA-R008:DTM13-12PA-R008
- J2: device SparkFun-Connectors:CONN_04SCREW -> SparkFun-Connectors:CONN_10"
Connections:
- removed net N$8: IC1.INT, U$1.25
- new net N$1: C5.1, F1.1, IC2.IN, J1.11
- new net N$26: IC1.INT, J2.8, U$1.25
- net GND: now also J1.1
- net N$14: now also J1.9; no longer J1.1
- net N$15: now also J1.7, J1.8; no longer J1.3, J1.5
- net N$16: now also J1.5; no longer J1.4
- net N$17: now also J1.4; no longer J1.2
- net N$20: now also F1.2, J1.12; no longer C5.1, IC2.IN, J2.1, J2.3
- net N$24: now also J1.2; no longer J2.4
- net N$25: now also J2.1, U$1.3.3V; no longer U$1.VIN
- net N$5: now also J2.3
- net N$6: now also J2.4
- net N$7: now also J2.7
- net N$9: now also J2.9
Other:
- moved on the sheet: R3
