File: Aeroneers/CAD Files/projects/FSAE NODE BOARD/node.sch (EAGLE design)
At the start: 24 parts, among them U1 DUAL-OPTOISOLATOR_SOIC8

Commit message: End of semester commit
Connections:
- net N$3: now also U$1.3.3V; no longer U$1.VIN
Changed lines of the file:
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@@
 <junction x="88.9" y="121.92"/>
 <wire x1="101.6" y1="106.68" x2="71.12" y2="106.68" width="0.1524" layer="91"/>
-<wire x1="71.12" y1="106.68" x2="71.12" y2="88.9" width="0.1524" layer="91"/>
-<pinref part="U$1" gate="G$1" pin="VIN"/>
-<wire x1="71.12" y1="88.9" x2="66.04" y2="88.9" width="0.1524" layer="91"/>
+<wire x1="71.12" y1="106.68" x2="71.12" y2="86.36" width="0.1524" layer="91"/>
 <pinref part="U$2" gate="G$1" pin="VCC"/>
 <wire x1="106.68" y1="83.82" x2="96.52" y2="83.82" width="0.1524" layer="91"/>
@@
 <junction x="-30.48" y="43.18"/>
 <wire x1="-30.48" y1="43.18" x2="-30.48" y2="2.54" width="0.1524" layer="91"/>
+<pinref part="U$1" gate="G$1" pin="3.3V"/>
+<wire x1="71.12" y1="86.36" x2="66.04" y2="86.36" width="0.1524" layer="91"/>
 </segment>
 </net>
